Commit message: robot xacro update

File: diff_drive/urdf/ddrive.gazebo.xacro (robot description, xacro)
@@ -1,10 +1,15 @@
 <?xml version="1.0"?>
 <robot name = "robot" xmlns:xacro="https://www.ros.org/wiki/xacro">
-<xacro:property name="base_size" value="1.0"/>
-<xacro:property name="wheel_r" value ="0.5"/>
+<xacro:property name="yaml_file" value="$(find diff_drive)/config/physical.yaml"/>
+<xacro:property name="params" value="${xacro.load_yaml(yaml_file)}"/>
+<xacro:property name="base_size" value="${params['/**']['ros__parameters']['base_size']}"/>
+<xacro:property name="length" value="${params['/**']['ros__parameters']['length']}"/>
+<xacro:property name="wheel_r" value="${params['/**']['ros__parameters']['wheel_r']}"/>
+<xacro:property name="wheel_l" value="${params['/**']['ros__parameters']['wheel_l']}"/>
+<xacro:property name="caster_r" value="${params['/**']['ros__parameters']['caster_r']}"/>
 <link name="base_link">
     <visual>
         <geometry>
-            <box size="${base_size} ${base_size} ${base_size}"/>
+            <box size="${length} ${base_size} ${base_size}"/>
         </geometry>
         <material name="blue_mat">
@@ -14,7 +19,117 @@
     <collision>
         <geometry>
-            <box size="${base_size} ${base_size} ${base_size}"/>
+            <box size="${length} ${base_size} ${base_size}"/>
         </geometry>
     </collision>
+    <inertial>
+        <mass value='5'/>
+        <inertia ixx='5.0' ixy='0' ixz='0' iyy='5.0' iyz='0' izz='3.0'/>
+    </inertial>
 </link>
+<link name = "left_wheel">
+    <visual>
+        <origin xyz="0 0 0" rpy="${pi/2} 0 0"/>
+        <geometry>
+            <cylinder radius="${wheel_r}" length="${wheel_l}"/>
+        </geometry>
+        <material name='red_mat'>
+            <color rgba = "1 0 0 0.8"/>
+        </material>
+    </visual>
+    <collision>
+        <origin xyz="0 0 0" rpy="${pi/2} 0 0"/>
+        <geometry>
+            <cylinder radius="${wheel_r}" length="${wheel_l}"/>
+        </geometry>
+    </collision>
+    <inertial>
+        <mass value='0.5'/>
+        <inertia ixx='0.01' ixy='0' ixz='0' iyy='0.02' iyz='0' izz='0.01'/>
+    </inertial>
+</link>
+<link name = "right_wheel">
+    <visual>
+        <origin xyz="0 0 0" rpy="${pi/2} 0 0"/>
+        <geometry>
+            <cylinder radius="${wheel_r}" length="${wheel_l}"/>
+        </geometry>
+        <material name='red_mat'>
+            <color rgba = "1 0 0 0.8"/>
+        </material>
+    </visual>
+    <collision>
+        <origin xyz="0 0 0" rpy="${pi/2} 0 0"/>
+        <geometry>
+            <cylinder radius="${wheel_r}" length="${wheel_l}"/>
+        </geometry>
+    </collision>
+    <inertial>
+        <mass value='0.5'/>
+        <inertia ixx='0.01' ixy='0' ixz='0' iyy='0.02' iyz='0' izz='0.01'/>
+    </inertial>
+</link>
+<link name="top_caster">
+    <visual>
+        <origin xyz="0 0 0" rpy="${pi/2} 0 0"/>
+        <geometry>
+            <sphere radius="${caster_r}"/>
+        </geometry>
+        <material name='green_mat'>
+            <color rgba = "0 1 0 1"/>
+        </material>
+    </visual>
+    <collision>
+        <origin xyz="0 0 0" rpy="${pi/2} 0 0"/>
+        <geometry>
+            <sphere radius="${caster_r}"/>
+        </geometry>
+    </collision>
+    <inertial>
+        <mass value='0.2'/>
+        <inertia ixx='0.001' ixy='0' ixz='0' iyy='0.001' iyz='0' izz='0.001'/>
+    </inertial>
+</link>
+<link name="bottom_caster">
+    <visual>
+        <origin xyz="0 0 0" rpy="${pi/2} 0 0"/>
+        <geometry>
+            <sphere radius="${caster_r}"/>
+        </geometry>
+        <material name='green_mat'>
+            <color rgba = "0 1 0 1"/>
+        </material>
+    </visual>
+    <collision>
+        <origin xyz="0 0 0" rpy="${pi/2} 0 0"/>
+        <geometry>
+            <sphere radius="${caster_r}"/>
+        </geometry>
+    </collision>
+    <inertial>
+        <mass value='0.2'/>
+        <inertia ixx='0.001' ixy='0' ixz='0' iyy='0.001' iyz='0' izz='0.001'/>
+    </inertial>
+</link>
+<joint name="base_l_wheel_joint" type="continuous">
+    <parent link="base_link"/>
+    <child link="left_wheel"/>
+    <origin xyz="${length/5} ${base_size/2} -${base_size/2}" rpy="0 0 0"/>
+    <axis xyz="0 1 0"/>
+</joint>
+<joint name="base_r_wheel_joint" type="continuous">
+    <parent link="base_link"/>
+    <child link="right_wheel"/>
+    <origin xyz="${length/5} -${base_size/2} -${base_size/2}" rpy="0 0 0"/>
+    <axis xyz="0 1 0"/>
+</joint>
+<joint name="base_top_caster_joint" type="fixed">
+  <parent link="base_link"/>
+  <child link="top_caster"/>
+  <origin xyz="-${length/2 - 2*caster_r} 0 ${base_size/2 + caster_r}" rpy="0 0 0"/>
+</joint>
+<joint name="base_bottom_caster_joint" type="fixed">
+  <parent link="base_link"/>
+  <child link="bottom_caster"/>
+  <origin xyz="-${length/2 - 2*caster_r} 0 -${base_size/2 + caster_r}" rpy="0 0 0"/>
+</joint>
 </robot>

Commit message: xacro urdf update

File: diff_drive/urdf/ddrive.gazebo.xacro (robot description, xacro)
@@ -1,135 +1,42 @@
 <?xml version="1.0"?>
 <robot name = "robot" xmlns:xacro="https://www.ros.org/wiki/xacro">
-<xacro:property name="yaml_file" value="$(find diff_drive)/config/physical.yaml"/>
-<xacro:property name="params" value="${xacro.load_yaml(yaml_file)}"/>
-<xacro:property name="base_size" value="${params['/**']['ros__parameters']['base_size']}"/>
-<xacro:property name="length" value="${params['/**']['ros__parameters']['length']}"/>
-<xacro:property name="wheel_r" value="${params['/**']['ros__parameters']['wheel_r']}"/>
-<xacro:property name="wheel_l" value="${params['/**']['ros__parameters']['wheel_l']}"/>
-<xacro:property name="caster_r" value="${params['/**']['ros__parameters']['caster_r']}"/>
-<link name="base_link">
-    <visual>
-        <geometry>
-            <box size="${length} ${base_size} ${base_size}"/>
-        </geometry>
-        <material name="blue_mat">
-            <color rgba="0 0 1 1"/>
+    <gazebo>
+        <plugin name="gz::sim::systems::DiffDrive" filename='gz-sim-diff-drive-system'>
+            <left_joint>base_l_wheel_joint</left_joint>
+            <right_joint>base_r_wheel_joint</right_joint>
+            <wheel_separation>${base_size}</wheel_separation>
+            <wheel_radius>${wheel_r}</wheel_radius>
+            <topic>/cmd_vel</topic>
+            <odom_topic>/odom</odom_topic>
+            <tf_topic>/tf</tf_topic>
+        </plugin>
+    </gazebo>
+    <gazebo>
+        <plugin name="gz::sim::systems::JointStatePublisher"
+                filename="gz-sim-joint-state-publisher-system">
+            <topic>/joint_states</topic>
+            <joint_name>base_l_wheel_joint</joint_name>
+            <joint_name>base_r_wheel_joint</joint_name>
+        </plugin>
+    </gazebo>
+    <gazebo reference="top_caster">
+        <mu1>0.0</mu1>
+        <mu2>0.0</mu2>
+        <material>
+            <ambient>0</ambient>
+            <diffuse>0</diffuse>
+            <specular>0</specular>
+            <emissive>0</emissive>
         </material>
-    </visual>
-    <collision>
-        <geometry>
-            <box size="${length} ${base_size} ${base_size}"/>
-        </geometry>
-    </collision>
-    <inertial>
-        <mass value='5'/>
-        <inertia ixx='5.0' ixy='0' ixz='0' iyy='5.0' iyz='0' izz='3.0'/>
-    </inertial>
-</link>
-<link name = "left_wheel">
-    <visual>
-        <origin xyz="0 0 0" rpy="${pi/2} 0 0"/>
-        <geometry>
-            <cylinder radius="${wheel_r}" length="${wheel_l}"/>
-        </geometry>
-        <material name='red_mat'>
-            <color rgba = "1 0 0 0.8"/>
+    </gazebo>
+    <gazebo reference="bottom_caster">
+        <mu1>0.0</mu1>
+        <mu2>0.0</mu2>
+        <material>
+            <ambient>0</ambient>
+            <diffuse>0</diffuse>
+            <specular>0</specular>
+            <emissive>0</emissive>
         </material>
-    </visual>
-    <collision>
-        <origin xyz="0 0 0" rpy="${pi/2} 0 0"/>
-        <geometry>
-            <cylinder radius="${wheel_r}" length="${wheel_l}"/>
-        </geometry>
-    </collision>
-    <inertial>
-        <mass value='0.5'/>
-        <inertia ixx='0.01' ixy='0' ixz='0' iyy='0.02' iyz='0' izz='0.01'/>
-    </inertial>
-</link>
-<link name = "right_wheel">
-    <visual>
-        <origin xyz="0 0 0" rpy="${pi/2} 0 0"/>
-        <geometry>
-            <cylinder radius="${wheel_r}" length="${wheel_l}"/>
-        </geometry>
-        <material name='red_mat'>
-            <color rgba = "1 0 0 0.8"/>
-        </material>
-    </visual>
-    <collision>
-        <origin xyz="0 0 0" rpy="${pi/2} 0 0"/>
-        <geometry>
-            <cylinder radius="${wheel_r}" length="${wheel_l}"/>
-        </geometry>
-    </collision>
-    <inertial>
-        <mass value='0.5'/>
-        <inertia ixx='0.01' ixy='0' ixz='0' iyy='0.02' iyz='0' izz='0.01'/>
-    </inertial>
-</link>
-<link name="top_caster">
-    <visual>
-        <origin xyz="0 0 0" rpy="${pi/2} 0 0"/>
-        <geometry>
-            <sphere radius="${caster_r}"/>
-        </geometry>
-        <material name='green_mat'>
-            <color rgba = "0 1 0 1"/>
-        </material>
-    </visual>
-    <collision>
-        <origin xyz="0 0 0" rpy="${pi/2} 0 0"/>
-        <geometry>
-            <sphere radius="${caster_r}"/>
-        </geometry>
-    </collision>
-    <inertial>
-        <mass value='0.2'/>
-        <inertia ixx='0.001' ixy='0' ixz='0' iyy='0.001' iyz='0' izz='0.001'/>
-    </inertial>
-</link>
-<link name="bottom_caster">
-    <visual>
-        <origin xyz="0 0 0" rpy="${pi/2} 0 0"/>
-        <geometry>
-            <sphere radius="${caster_r}"/>
-        </geometry>
-        <material name='green_mat'>
-            <color rgba = "0 1 0 1"/>
-        </material>
-    </visual>
-    <collision>
-        <origin xyz="0 0 0" rpy="${pi/2} 0 0"/>
-        <geometry>
-            <sphere radius="${caster_r}"/>
-        </geometry>
-    </collision>
-    <inertial>
-        <mass value='0.2'/>
-        <inertia ixx='0.001' ixy='0' ixz='0' iyy='0.001' iyz='0' izz='0.001'/>
-    </inertial>
-</link>
-<joint name="base_l_wheel_joint" type="continuous">
-    <parent link="base_link"/>
-    <child link="left_wheel"/>
-    <origin xyz="${length/5} ${base_size/2} -${base_size/2}" rpy="0 0 0"/>
-    <axis xyz="0 1 0"/>
-</joint>
-<joint name="base_r_wheel_joint" type="continuous">
-    <parent link="base_link"/>
-    <child link="right_wheel"/>
-    <origin xyz="${length/5} -${base_size/2} -${base_size/2}" rpy="0 0 0"/>
-    <axis xyz="0 1 0"/>
-</joint>
-<joint name="base_top_caster_joint" type="fixed">
-  <parent link="base_link"/>
-  <child link="top_caster"/>
-  <origin xyz="-${length/2 - 2*caster_r} 0 ${base_size/2 + caster_r}" rpy="0 0 0"/>
-</joint>
-<joint name="base_bottom_caster_joint" type="fixed">
-  <parent link="base_link"/>
-  <child link="bottom_caster"/>
-  <origin xyz="-${length/2 - 2*caster_r} 0 -${base_size/2 + caster_r}" rpy="0 0 0"/>
-</joint>
+    </gazebo>
 </robot>

Commit message: fixed topic mismatch

File: diff_drive/urdf/ddrive.gazebo.xacro (robot description, xacro)
@@ -7,6 +7,5 @@
             <wheel_separation>${base_size}</wheel_separation>
             <wheel_radius>${wheel_r}</wheel_radius>
-            <topic>cmd_vel</topic>
-            <odom_topic>odom</odom_topic>
+            <topic>/model/robot/cmd_vel</topic>
         </plugin>
     </gazebo>

File: diff_drive/urdf/ddrive.urdf.xacro (robot description, xacro)
@@ -118,5 +118,5 @@
     <parent link="base_link"/>
     <child link="left_wheel"/>
-    <origin xyz="${length/5} ${base_size/2} -${base_size/2}" rpy="0 0 0"/>
+    <origin xyz="0 ${base_size/2+wheel_l} 0" rpy="0 0 0"/>
     <axis xyz="0 1 0"/>
 </joint>
@@ -124,13 +124,13 @@
     <parent link="base_link"/>
     <child link="right_wheel"/>
-    <origin xyz="${length/5} -${base_size/2} -${base_size/2}" rpy="0 0 0"/>
+    <origin xyz="0 -${base_size/2+wheel_l} 0" rpy="0 0 0"/>
     <axis xyz="0 1 0"/>
 </joint>
-<joint name="base_top_caster_joint" type="fixed">
+<joint name="base_top_caster_joint" type="continuous">
   <parent link="base_link"/>
   <child link="top_caster"/>
   <origin xyz="-${length/2 - 2*caster_r} 0 ${base_size/2 + caster_r}" rpy="0 0 0"/>
 </joint>
-<joint name="base_bottom_caster_joint" type="fixed">
+<joint name="base_bottom_caster_joint" type="continuous">
   <parent link="base_link"/>
   <child link="bottom_caster"/>

Commit message: update xacro

File: diff_drive/urdf/ddrive.gazebo.xacro (robot description, xacro)
@@ -8,4 +8,6 @@
             <wheel_radius>${wheel_r}</wheel_radius>
             <topic>/model/robot/cmd_vel</topic>
+            <topic>/model/robot/tf</topic>
+            <topic>/model/robot/odom</topic>
         </plugin>
     </gazebo>

File: diff_drive/urdf/ddrive.urdf.xacro (robot description, xacro)
@@ -4,4 +4,5 @@
 <xacro:property name="params" value="${xacro.load_yaml(yaml_file)}"/>
 <xacro:property name="base_size" value="${params['/**']['ros__parameters']['base_size']}"/>
+<xacro:property name="width" value="${params['/**']['ros__parameters']['width']}"/>
 <xacro:property name="length" value="${params['/**']['ros__parameters']['length']}"/>
 <xacro:property name="wheel_r" value="${params['/**']['ros__parameters']['wheel_r']}"/>
@@ -15,5 +16,5 @@
     <visual>
         <geometry>
-            <box size="${length} ${base_size} ${base_size}"/>
+            <box size="${length} ${base_size} ${width}"/>
         </geometry>
         <material name="blue_mat">
@@ -23,5 +24,5 @@
     <collision>
         <geometry>
-            <box size="${length} ${base_size} ${base_size}"/>
+            <box size="${length} ${base_size} ${width}"/>
         </geometry>
     </collision>
@@ -118,5 +119,5 @@
     <parent link="base_link"/>
     <child link="left_wheel"/>
-    <origin xyz="0 ${base_size/2+wheel_l} 0" rpy="0 0 0"/>
+    <origin xyz="${width*3/2} ${base_size/2+wheel_l} 0" rpy="0 0 0"/>
     <axis xyz="0 1 0"/>
 </joint>
@@ -124,5 +125,5 @@
     <parent link="base_link"/>
     <child link="right_wheel"/>
-    <origin xyz="0 -${base_size/2+wheel_l} 0" rpy="0 0 0"/>
+    <origin xyz="${width*3/2} -${base_size/2+wheel_l} 0" rpy="0 0 0"/>
     <axis xyz="0 1 0"/>
 </joint>
@@ -130,10 +131,10 @@
   <parent link="base_link"/>
   <child link="top_caster"/>
-  <origin xyz="-${length/2 - 2*caster_r} 0 ${base_size/2 + caster_r}" rpy="0 0 0"/>
+  <origin xyz="-${length/2 - 2*caster_r} 0 ${width/2 + caster_r}" rpy="0 0 0"/>
 </joint>
 <joint name="base_bottom_caster_joint" type="continuous">
   <parent link="base_link"/>
   <child link="bottom_caster"/>
-  <origin xyz="-${length/2 - 2*caster_r} 0 -${base_size/2 + caster_r}" rpy="0 0 0"/>
+  <origin xyz="-${length/2 - 2*caster_r} 0 -${width/2 + caster_r}" rpy="0 0 0"/>
 </joint>
 </robot>

Commit message: minor error fixes

File: diff_drive/urdf/ddrive.gazebo.xacro (robot description, xacro)
@@ -23,20 +23,8 @@
         <mu1>0.0</mu1>
         <mu2>0.0</mu2>
-        <material>
-            <ambient>0</ambient>
-            <diffuse>0</diffuse>
-            <specular>0</specular>
-            <emissive>0</emissive>
-        </material>
     </gazebo>
     <gazebo reference="bottom_caster">
         <mu1>0.0</mu1>
         <mu2>0.0</mu2>
-        <material>
-            <ambient>0</ambient>
-            <diffuse>0</diffuse>
-            <specular>0</specular>
-            <emissive>0</emissive>
-        </material>
     </gazebo>
 </robot>
