Commit message: move robot

File: diff_drive/urdf/ddrive.urdf.xacro (robot description, xacro)
@@ -29,5 +29,5 @@
     <inertial>
         <mass value='5'/>
-        <inertia ixx='5.0' ixy='0' ixz='0' iyy='5.0' iyz='0' izz='3.0'/>
+        <inertia ixx='0.521' ixy='0' ixz='0' iyy='3.854' iyz='0' izz='4.167'/>
     </inertial>
 </link>
@@ -49,6 +49,6 @@
     </collision>
     <inertial>
-        <mass value='0.5'/>
-        <inertia ixx='0.01' ixy='0' ixz='0' iyy='0.02' iyz='0' izz='0.01'/>
+        <mass value='3'/>
+        <inertia ixx='0.28' ixy='0' ixz='0' iyy='0.54' iyz='0' izz='0.28'/>
     </inertial>
 </link>
@@ -70,6 +70,6 @@
     </collision>
     <inertial>
-        <mass value='0.5'/>
-        <inertia ixx='0.01' ixy='0' ixz='0' iyy='0.02' iyz='0' izz='0.01'/>
+        <mass value='3'/>
+        <inertia ixx='0.28' ixy='0' ixz='0' iyy='0.54' iyz='0' izz='0.28'/>
     </inertial>
 </link>
@@ -91,6 +91,6 @@
     </collision>
     <inertial>
-        <mass value='0.2'/>
-        <inertia ixx='0.001' ixy='0' ixz='0' iyy='0.001' iyz='0' izz='0.001'/>
+        <mass value='1.0'/>
+        <inertia ixx='0.016' ixy='0' ixz='0' iyy='0.016' iyz='0' izz='0.016'/>
     </inertial>
 </link>
@@ -112,6 +112,6 @@
     </collision>
     <inertial>
-        <mass value='0.2'/>
-        <inertia ixx='0.001' ixy='0' ixz='0' iyy='0.001' iyz='0' izz='0.001'/>
+        <mass value='1.0'/>
+        <inertia ixx='0.016' ixy='0' ixz='0' iyy='0.016' iyz='0' izz='0.016'/>
     </inertial>
 </link>
@@ -132,4 +132,5 @@
   <child link="top_caster"/>
   <origin xyz="-${length/2 - 2*caster_r} 0 ${width/2 + caster_r}" rpy="0 0 0"/>
+  <axis xyz="0 1 0"/>
 </joint>
 <joint name="base_bottom_caster_joint" type="continuous">
@@ -137,4 +138,5 @@
   <child link="bottom_caster"/>
   <origin xyz="-${length/2 - 2*caster_r} 0 -${width/2 + caster_r}" rpy="0 0 0"/>
+  <axis xyz="0 1 0"/>
 </joint>
 </robot>

Commit message: finishing up

File: diff_drive/urdf/ddrive.urdf.xacro (robot description, xacro)
@@ -29,5 +29,5 @@
     <inertial>
         <mass value='5'/>
-        <inertia ixx='0.521' ixy='0' ixz='0' iyy='3.854' iyz='0' izz='4.167'/>
+        <inertia ixx='0.02' ixy='0' ixz='0' iyy='0.15' iyz='0' izz='0.16'/>
     </inertial>
 </link>
@@ -50,5 +50,5 @@
     <inertial>
         <mass value='3'/>
-        <inertia ixx='0.28' ixy='0' ixz='0' iyy='0.54' iyz='0' izz='0.28'/>
+        <inertia ixx='0.011' ixy='0' ixz='0' iyy='0.02' iyz='0' izz='0.01'/>
     </inertial>
 </link>
@@ -71,5 +71,5 @@
     <inertial>
         <mass value='3'/>
-        <inertia ixx='0.28' ixy='0' ixz='0' iyy='0.54' iyz='0' izz='0.28'/>
+        <inertia ixx='0.011' ixy='0' ixz='0' iyy='0.02' iyz='0' izz='0.01'/>
     </inertial>
 </link>
@@ -91,6 +91,6 @@
     </collision>
     <inertial>
-        <mass value='1.0'/>
-        <inertia ixx='0.016' ixy='0' ixz='0' iyy='0.016' iyz='0' izz='0.016'/>
+        <mass value='0.2'/>
+        <inertia ixx='0.000128' ixy='0' ixz='0' iyy='0.000128' iyz='0' izz='0.000128'/>
     </inertial>
 </link>
@@ -112,6 +112,6 @@
     </collision>
     <inertial>
-        <mass value='1.0'/>
-        <inertia ixx='0.016' ixy='0' ixz='0' iyy='0.016' iyz='0' izz='0.016'/>
+        <mass value='0.2'/>
+        <inertia ixx='0.000128' ixy='0' ixz='0' iyy='0.000128' iyz='0' izz='0.000128'/>
     </inertial>
 </link>
@@ -119,5 +119,5 @@
     <parent link="base_link"/>
     <child link="left_wheel"/>
-    <origin xyz="${width*3/2} ${base_size/2+wheel_l} 0" rpy="0 0 0"/>
+    <origin xyz="${length/2} ${base_size/2+wheel_l} 0" rpy="0 0 0"/>
     <axis xyz="0 1 0"/>
 </joint>
@@ -125,5 +125,5 @@
     <parent link="base_link"/>
     <child link="right_wheel"/>
-    <origin xyz="${width*3/2} -${base_size/2+wheel_l} 0" rpy="0 0 0"/>
+    <origin xyz="${length/2} -${base_size/2+wheel_l} 0" rpy="0 0 0"/>
     <axis xyz="0 1 0"/>
 </joint>

Commit message: Graded

File: diff_drive/urdf/ddrive.urdf.xacro (robot description, xacro)
@@ -28,5 +28,6 @@
     </collision>
     <inertial>
-        <mass value='5'/>
+      <mass value='5'/>
+      <!-- should be using formulas for the inertia based on the parameters-->
         <inertia ixx='0.02' ixy='0' ixz='0' iyy='0.15' iyz='0' izz='0.16'/>
     </inertial>
